File: Board/Timer-Ruler_CR2032_on_bottom.sch (EAGLE design)
At the start: 33 parts, among them U1 ATMEGA328P_TQFP, Y1 8MHZ

Commit message: update
Parts:
- B0, B2, SCL, SDA: value (none) -> nur PAD, keine Stiftleiste
- JP1: value ISP -> nur PAD, keine Stiftleiste
Changed lines of the file:
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@@
 <part name="S2" library="Wurth_Elektronik_Electromechanic_Switchs_rev15b" deviceset="431151015826" device=""/>
 <part name="S3" library="Wurth_Elektronik_Electromechanic_Switchs_rev15b" deviceset="431151015826" device=""/>
-<part name="JP1" library="pinhead" deviceset="PINHD-2X3" device="" value="ISP"/>
+<part name="JP1" library="pinhead" deviceset="PINHD-2X3" device="" value="nur PAD, keine Stiftleiste"/>
 <part name="GND3" library="supply1" deviceset="GND" device=""/>
 <part name="P+2" library="supply1" deviceset="VCC" device=""/>
@@
 <part name="P+1" library="supply1" deviceset="VCC" device=""/>
 <part name="Y1" library="SparkFun-FreqCtrl" deviceset="RESONATOR" device="8MHZ" value="8MHZ"/>
-<part name="SDA" library="pinhead" deviceset="PINHD-1X1" device=""/>
-<part name="SCL" library="pinhead" deviceset="PINHD-1X1" device=""/>
+<part name="SDA" library="pinhead" deviceset="PINHD-1X1" device="" value="nur PAD, keine Stiftleiste"/>
+<part name="SCL" library="pinhead" deviceset="PINHD-1X1" device="" value="nur PAD, keine Stiftleiste"/>
 <part name="U$3" library="Ava" deviceset="RENATA_STMU2032" device=""/>
 <part name="U$4" library="Ava" deviceset="C+K_AYZ0202AGRLC" device=""/>
-<part name="B0" library="pinhead" deviceset="PINHD-1X1" device=""/>
-<part name="B2" library="pinhead" deviceset="PINHD-1X1" device=""/>
+<part name="B0" library="pinhead" deviceset="PINHD-1X1" device="" value="nur PAD, keine Stiftleiste"/>
+<part name="B2" library="pinhead" deviceset="PINHD-1X1" device="" value="nur PAD, keine Stiftleiste"/>
 </parts>
 <sheets>
@@
 </sheet>
 </sheets>
+<errors>
+</errors>
 </schematic>
 </drawing>
