File: Board/Timer-Ruler_CR2032_on_top.brd (EAGLE design)
At the start: 100 x 80 mm, 33 parts, among them U1 ATMEGA328P_TQFP, Y1 8MHZ

Commit message: update
Parts:
- B0, B2, SCL, SDA: value (none) -> nur PAD, keine Stiftleiste
Changed lines of the file:
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@@
 <text x="30.48" y="20.955" size="1.778" layer="25" font="vector" rot="SR270" align="center">T2</text>
 <text x="30.48" y="13.97" size="1.778" layer="25" font="vector" rot="SR270" align="center">T3</text>
-<text x="33.441428125" y="38.190725" size="1.016" layer="25" font="vector" align="center">1</text>
+<text x="41.696428125" y="43.270725" size="1.016" layer="25" font="vector" align="center">1</text>
 <text x="64.135" y="41.275" size="0.889" layer="26" font="vector" rot="MR0" align="top-left">TimeR Rev.1
 01/2016@AE</text>
-<dimension x1="20.955" y1="44.45" x2="66.04" y2="45.72" x3="43.4975" y3="46.99" textsize="1.778" layer="1" dtype="horizontal"/>
-<dimension x1="20.955" y1="44.45" x2="19.05" y2="10.16" x3="17.78" y3="27.305" textsize="1.778" layer="1" dtype="vertical"/>
+<dimension x1="20.955" y1="44.45" x2="66.04" y2="45.72" x3="43.4975" y3="46.99" textsize="1.778" layer="20" dtype="horizontal"/>
+<dimension x1="20.955" y1="44.45" x2="19.05" y2="10.16" x3="17.78" y3="27.305" textsize="1.778" layer="20" dtype="vertical"/>
 </plain>
 <attributes>
@@
 <element name="S3" library="Wurth_Elektronik_Electromechanic_Switchs_rev15b" package="431181015816" value="431151015826" x="25.4" y="13.97" smashed="yes" rot="R180"/>
 <element name="JP1" library="pinhead" package="2X03" value="ISP" x="36.83" y="41.275" smashed="yes" rot="R180">
-<attribute name="VALUE" x="43.815" y="43.815" size="1.27" layer="27" rot="R180"/>
+<attribute name="VALUE" x="44.45" y="40.64" size="1.27" layer="27" rot="R180"/>
 </element>
 <element name="R10" library="resistor" package="R0402" value="220R" x="32.135" y="41.877775" smashed="yes" rot="R270"/>
@@
 <attribute name="PROD_ID" value="XTAL-08895" x="41.91" y="25.4" size="1.778" layer="27" rot="R45" display="off"/>
 </element>
-<element name="SDA" library="pinhead" package="1X01" value="" x="22.86" y="35.56" smashed="yes">
-<attribute name="NAME" x="24.6888" y="34.8488" size="1.27" layer="25" ratio="10"/>
-<attribute name="VALUE" x="21.59" y="32.385" size="1.27" layer="27"/>
-</element>
-<element name="SCL" library="pinhead" package="1X01" value="" x="22.86" y="33.02" smashed="yes" rot="R90">
-<attribute name="NAME" x="24.8412" y="32.3088" size="1.27" layer="25" ratio="10"/>
-<attribute name="VALUE" x="26.035" y="31.75" size="1.27" layer="27" rot="R90"/>
+<element name="SDA" library="pinhead" package="1X01" value="nur PAD, keine Stiftleiste" x="22.86" y="35.56" smashed="yes">
+<attribute name="NAME" x="24.6888" y="35.4838" size="1.27" layer="25" ratio="10" align="center-left"/>
+</element>
+<element name="SCL" library="pinhead" package="1X01" value="nur PAD, keine Stiftleiste" x="22.86" y="33.02" smashed="yes" rot="R90">
+<attribute name="NAME" x="24.8412" y="32.9438" size="1.27" layer="25" ratio="10" align="center-left"/>
 </element>
 <element name="U$3" library="Ava" package="SMTU2032" value="RENATA_STMU2032" x="54.61" y="29.845" smashed="yes" rot="R125.6"/>
 <element name="U$4" library="Ava" package="C+K_AYZ0202AGRLC" value="C+K_AYZ0202AGRLC" x="25.4" y="40.64" rot="R180"/>
-<element name="B0" library="pinhead" package="1X01" value="" x="57.785" y="42.545" smashed="yes">
+<element name="B0" library="pinhead" package="1X01" value="nur PAD, keine Stiftleiste" x="57.785" y="42.545" smashed="yes">
 <attribute name="NAME" x="61.6712" y="43.2562" size="1.27" layer="25" ratio="10" rot="R180"/>
-<attribute name="VALUE" x="56.515" y="39.37" size="1.27" layer="27"/>
-</element>
-<element name="B2" library="pinhead" package="1X01" value="" x="55.245" y="42.545" smashed="yes">
+</element>
+<element name="B2" library="pinhead" package="1X01" value="nur PAD, keine Stiftleiste" x="55.245" y="42.545" smashed="yes">
 <attribute name="NAME" x="51.5112" y="43.2562" size="1.27" layer="25" ratio="10" rot="R180" align="bottom-right"/>
-<attribute name="VALUE" x="53.975" y="39.37" size="1.27" layer="27"/>
 </element>
 </elements>
@@
 <wire x1="26.075" y1="26.09" x2="25.4" y2="25.415" width="0.4064" layer="1"/>
 <wire x1="49.53" y1="14.19" x2="52.07" y2="14.19" width="0.4064" layer="1"/>
-<wire x1="33.02" y1="14.19" x2="31.285" y2="12.12" width="0.4064" layer="1"/>
 <wire x1="31.285" y1="12.12" x2="27.7" y2="12.12" width="0.4064" layer="1"/>
 <wire x1="27.7" y1="19.105" x2="27.305" y2="18.71" width="0.4064" layer="1"/>
@@
 <wire x1="26.075" y1="26.09" x2="26.67" y2="26.09" width="0.4064" layer="1"/>
 <wire x1="26.67" y1="26.09" x2="27.7" y2="26.09" width="0.4064" layer="1"/>
-<wire x1="26.035" y1="32.385" x2="26.67" y2="31.75" width="0.4064" layer="1"/>
 <wire x1="26.67" y1="31.75" x2="26.67" y2="26.09" width="0.4064" layer="1"/>
 <wire x1="34.29" y1="40.005" x2="34.29" y2="33.02" width="0.4064" layer="16"/>
@@
 <wire x1="39.016796875" y1="27.86614375" x2="40.14816875" y2="28.997515625" width="0" layer="19" extent="1-1"/>
 <wire x1="25.4" y1="37.815" x2="25.4" y2="33.02" width="0.4064" layer="1"/>
-<wire x1="25.4" y1="33.02" x2="26.035" y2="32.385" width="0.4064" layer="1"/>
+<wire x1="25.4" y1="33.02" x2="26.67" y2="31.75" width="0.4064" layer="1"/>
+<wire x1="31.285" y1="12.12" x2="31.285" y2="12.455" width="0.4064" layer="1"/>
+<wire x1="31.285" y1="12.455" x2="33.02" y2="14.19" width="0.4064" layer="1"/>
 </signal>
 <signal name="LED1">
@@
 <wire x1="35.208884375" y1="36.1995375" x2="39.37" y2="32.038421875" width="0.4064" layer="1"/>
 <wire x1="39.37" y1="32.038421875" x2="39.37" y2="31.75" width="0.4064" layer="1"/>
-<wire x1="35.208884375" y1="36.1995375" x2="33.9211625" y2="37.46278125" width="0.4064" layer="1"/>
-<wire x1="33.9211625" y1="37.46278125" x2="32.385" y2="37.465" width="0.4064" layer="1"/>
 <wire x1="32.385" y1="37.465" x2="32.385" y2="40.977775" width="0.4064" layer="1"/>
 <wire x1="32.385" y1="40.977775" x2="32.135" y2="41.227775" width="0.4064" layer="1"/>
@@
 <wire x1="38.735" y1="29.21" x2="39.513171875" y2="28.431828125" width="0.4064" layer="1"/>
 <wire x1="39.513171875" y1="28.431828125" x2="39.58248125" y2="28.431828125" width="0.4064" layer="1"/>
+<wire x1="32.385" y1="37.465" x2="33.943421875" y2="37.465" width="0.4064" layer="1"/>
+<wire x1="33.943421875" y1="37.465" x2="35.208884375" y2="36.1995375" width="0.4064" layer="1"/>
 </signal>
 <signal name="MOSI">
 <contactref element="U1" pad="15"/>
 <contactref element="JP1" pad="4"/>
-<wire x1="36.83" y1="40.005" x2="37.465" y2="40.005" width="0.4064" layer="16"/>
-<wire x1="37.465" y1="40.005" x2="39.462403125" y2="37.776540625" width="0.4064" layer="16"/>
 <via x="39.462403125" y="37.776540625" extent="1-16" drill="0.6" shape="square"/>
-<wire x1="39.462403125" y1="37.776540625" x2="39.716575" y2="37.465" width="0.4064" layer="1"/>
-<wire x1="39.716575" y1="37.465" x2="38.4511125" y2="36.1995375" width="0.4064" layer="1"/>
+<wire x1="39.462403125" y1="37.776540625" x2="39.058459375" y2="37.776540625" width="0.4064" layer="16"/>
+<wire x1="39.058459375" y1="37.776540625" x2="36.83" y2="40.005" width="0.4064" layer="16"/>
+<wire x1="39.462403125" y1="37.776540625" x2="39.462403125" y2="37.210828125" width="0.4064" layer="1"/>
+<wire x1="39.462403125" y1="37.210828125" x2="38.4511125" y2="36.1995375" width="0.4064" layer="1"/>
 </signal>
 <signal name="RST">
